File: hardware/OPNpool r3.brd (EAGLE design)
At the start: 63 x 58 mm, 16 parts, among them J2 RS485-TERM-SPTAF, J3 ESP-JTAG-2X05, SW1 Factory (5 sec), U1 MAX3485CSA+

Commit message: routed pcb r3
Parts:
- PCB1: device Coert Vonk:LOLIN-D32 -> Coert-Vonk:LOLIN-D32
- moved PCB1 0.49 mm to (39.0, 30.0)
Routing:
- net A: track 0.00 -> 95.2 mm, vias 0 -> 3
- net B: track 0.00 -> 92.7 mm, vias 0 -> 1
- net 3V3: track 0.00 -> 83.5 mm, vias 0 -> 1
- net JTAG_!RST: track 0.00 -> 67.1 mm, vias 0 -> 1
- net TX: track 0.00 -> 58.6 mm, vias 0 -> 2
- net RX2: track 0.00 -> 52.0 mm, vias 0 -> 2
- net N$3: track 0.00 -> 50.1 mm
- net RTS: track 0.00 -> 43.6 mm, vias 0 -> 1
- net JTAG_MS: track 0.00 -> 36.5 mm
- net JTAG_CK: track 0.00 -> 35.5 mm
- net JTAG_DI: track 0.00 -> 32.4 mm
- net VOUT: track 0.00 -> 23.1 mm
- net 15V: track 0.00 -> 19.3 mm
- net VIN: track 0.00 -> 14.1 mm
- net JTAG_DO: track 0.00 -> 7.27 mm
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